Commit message: Added blade to the mock cutting plate urdf, but collisions still need to be handled Cleaned up old commented code from stock handler

File: ram_support/urdf/xacros/cutting_plate.xacro (robot description, xacro)
@@ -16,5 +16,18 @@
       </collision>
     </link>
-    <link name="cutting_tool_base"/>
+    <link name="cutting_tool_base">
+      <visual>
+        <origin xyz="0 0 -0.25" rpy="0 0 0"/>
+        <geometry>
+          <mesh filename="package://ram_support/meshes/tools/visual/mock_cutting_blade.dae"/>
+        </geometry>
+      </visual>
+      <collision>
+        <origin xyz="0 0 -0.25" rpy="0 0 0"/>
+        <geometry>
+          <mesh filename="package://ram_support/meshes/tools/collision/mock_cutting_blade.stl"/>
+        </geometry>
+      </collision>
+    </link>
     <joint name="cutting_plate_tool_joint" type="fixed">
       <parent link="cutting_plate"/>

Commit message: Updated to DUK8 blade that has been quoted for. Changed the cutting plate setup to make blade changes easier. updated toolpath follower for new collison object name. added half mm rise to tool path allowing planning near the base of the cutting plate

File: ram_support/urdf/xacros/cutting_plate.xacro (robot description, xacro)
@@ -16,29 +16,42 @@
       </collision>
     </link>
-    <link name="cutting_tool_base">
+    <joint name="cutting_plate_surface_joint" type="fixed">
+      <parent link="cutting_plate"/>
+      <child link="cutting_plate_base"/>
+      <origin xyz="0 0 0.25" rpy="0 0 0"/>
+    </joint>
+    <link name="cutting_plate_base"/>
+  <!-- Cutting tool selected-->
+    <link name="cutting_tool">
       <visual>
-        <origin xyz="0 0 -0.25" rpy="0 0 0"/>
+        <origin xyz="0 0 0" rpy="0 0 0"/>
         <geometry>
-          <mesh filename="package://ram_support/meshes/tools/visual/mock_cutting_blade.dae"/>
+          <mesh filename="package://ram_support/meshes/tools/visual/DUK8.dae"/>
         </geometry>
       </visual>
       <collision>
-        <origin xyz="0 0 -0.25" rpy="0 0 0"/>
+        <origin xyz="0 0 0" rpy="0 0 0"/>
         <geometry>
-          <mesh filename="package://ram_support/meshes/tools/collision/mock_cutting_blade.stl"/>
+          <mesh filename="package://ram_support/meshes/tools/collision/DUK8.stl"/>
         </geometry>
       </collision>
     </link>
-    <joint name="cutting_plate_tool_joint" type="fixed">
-      <parent link="cutting_plate"/>
+    <link name="cutting_tool_base"/>
+    <link name="cutting_tool_tip"/>
+    <joint name="cutting_tool_joint" type="fixed">
+      <parent link="cutting_plate_base"/>
+      <child link="cutting_tool"/>
+      <origin xyz="0 0 -0.0035" rpy="0 0 0"/>
+    </joint>
+    <joint name="cutting_tool_base_joint" type="fixed">
+      <parent link="cutting_tool"/>
       <child link="cutting_tool_base"/>
-      <origin xyz="0 0 0.25" rpy="0 0 0"/>
+      <origin xyz="-0.003152 0 0.0035" rpy="0 0 0"/>
     </joint>
-    <joint name="cutting_tool_base_tip" type="fixed">
-      <parent link="cutting_tool_base"/>
+    <joint name="cutting_tool_tip_joint" type="fixed">
+      <parent link="cutting_tool"/>
       <child link="cutting_tool_tip"/>
-      <origin xyz="0 0 0.014158" rpy="0 0 0"/>
+      <origin xyz="0 0 0.0087" rpy="0 0 0"/>
     </joint>
-    <link name="cutting_tool_tip"/>
   </xacro:macro>
 </robot>
