Commit message: basic stock handler now working, allowing the stock to be loaded and unloaded from the planning scene, then attached and detached from a named link. Currently using default params, as the yaml file will not load. toolpath handler can now display the markers, seems to be from changing the reference frame to gripper_jaw_centre but unsure why that is. updated PGN-80 urdf with links for the gripper jaws and fixed error in joint limit on the gripper.

File: ram_support/urdf/xacros/schunk_gripper_pgn_80.xacro (robot description, xacro)
@@ -22,5 +22,5 @@
       <child link="${robot_name}_link_left"/>
       <origin xyz="0 0 0.0" rpy="0 0 0"/>
-      <limit lower="0.000" upper="0.005"
+      <limit lower="0.000" upper="0.004"
              effort="${max_effort}" velocity="0.0833" />
     </joint>
@@ -45,5 +45,5 @@
       <origin xyz="0 0 0" rpy="0 0 ${pi}"/>
       <axis xyz="1 0 0"/>
-      <limit lower="0.000" upper="0.005"
+      <limit lower="0.000" upper="0.004"
              effort="${max_effort}" velocity="0.0833" />
       <mimic joint="${robot_name}_joint_left"/>
@@ -63,4 +63,22 @@
       </collision>
     </link>
+    <link name="${robot_name}_jaw_centre"/>
+    <joint name="${robot_name}_jaw_centre_joint" type="fixed">
+      <parent link="${robot_name}_link_main_body"/>
+      <child link="${robot_name}_jaw_centre"/>
+      <origin xyz="0 0 0.078850" rpy="0 0 0"/>
+    </joint>
+    <link name="${robot_name}_jaw_left"/>
+    <joint name="${robot_name}_jaw_left_joint" type="fixed">
+      <parent link="${robot_name}_link_left"/>
+      <child link="${robot_name}_jaw_left"/>
+      <origin xyz="0.000524 0 0.078850" rpy="0 0 0"/>
+    </joint>
+    <link name="${robot_name}_jaw_right"/>
+    <joint name="${robot_name}_jaw_right_joint" type="fixed">
+      <parent link="${robot_name}_link_right"/>
+      <child link="${robot_name}_jaw_right"/>
+      <origin xyz="0.000524 0 0.078850" rpy="0 0 ${pi}"/>
+    </joint>
     <transmission name="${robot_name}_tran_right">
       <type>transmission_interface/SimpleTransmission</type>

Commit message: Moved iiwa and gripper to ros2 control fake components both working well.

File: ram_support/urdf/xacros/schunk_gripper_pgn_80.xacro (robot description, xacro)
@@ -47,5 +47,5 @@
       <limit lower="0.000" upper="0.004"
              effort="${max_effort}" velocity="0.0833" />
-      <mimic joint="${robot_name}_joint_left"/>
+<!--      <mimic joint="${robot_name}_joint_left"/>-->
     </joint>
     <link name="${robot_name}_link_right">
@@ -81,24 +81,6 @@
       <origin xyz="0.000524 0 0.078850" rpy="0 0 ${pi}"/>
     </joint>
-    <transmission name="${robot_name}_tran_right">
-      <type>transmission_interface/SimpleTransmission</type>
-      <joint name="${robot_name}_joint_right">
-	<hardwareInterface>hardware_interface/${hardware_interface}</hardwareInterface>
-      </joint>
-      <actuator name="${robot_name}_motor_right">
-	<hardwareInterface>hardware_interface/${hardware_interface}</hardwareInterface>
-	<mechanicalReduction>1</mechanicalReduction>
-      </actuator>
-    </transmission>
-    <transmission name="${robot_name}_tran_left">
-      <type>transmission_interface/SimpleTransmission</type>
-      <joint name="${robot_name}_joint_left">
-	<hardwareInterface>hardware_interface/${hardware_interface}</hardwareInterface>
-      </joint>
-      <actuator name="${robot_name}_motor_left">
-	<hardwareInterface>hardware_interface/${hardware_interface}</hardwareInterface>
-	<mechanicalReduction>1</mechanicalReduction>
-      </actuator>
-    </transmission>
+    <xacro:include filename="$(find ram_support)/urdf/xacros/control/gripper.ros2_control.xacro" />
+    <xacro:gripper_interface name="${robot_name}"/>
   </xacro:macro>
 </robot>

Commit message: implant holder configured for planning, stock handler allows for touch links to be set as params on start, implant support collision mesh in the xacro has been commented out

File: ram_support/urdf/xacros/schunk_gripper_pgn_80.xacro (robot description, xacro)
@@ -67,10 +67,10 @@
         </geometry>
       </visual>
-      <collision>
-        <origin xyz="0 0 0" rpy="0 0 0"/>
-        <geometry>
-          <mesh filename="package://ram_support/meshes/schunk_gripper/pgn_80/collision/implant_support.stl" />
-        </geometry>
-      </collision>
+<!--      <collision>-->
+<!--        <origin xyz="0 0 0" rpy="0 0 0"/>-->
+<!--        <geometry>-->
+<!--          <mesh filename="package://ram_support/meshes/schunk_gripper/pgn_80/collision/implant_support.stl" />-->
+<!--        </geometry>-->
+<!--      </collision>-->
     </link>
     <!-- joint between main body and left jaw -->
