Commit message: added fingers for the gripper and the large medpor implant, changed gripper joint to mimic each other

File: ram_support/urdf/mock_iiwa_workcell.urdf.xacro (robot description, xacro)
@@ -10,4 +10,6 @@
     <xacro:include filename="$(find ram_support)/urdf/xacros/milling_plate.xacro"/>
     <xacro:include filename="$(find ram_support)/urdf/xacros/cutting_plate.xacro"/>
+    <xacro:include filename="$(find ram_support)/urdf/xacros/implant_grasp_fingers.xacro"/>
+    <xacro:include filename="$(find ram_support)/urdf/xacros/medpor_stock.xacro"/>
     <xacro:arg name="iiwa_name" default="iiwa"/>
     <xacro:arg name="gripper_name" default="gripper"/>
@@ -39,4 +41,5 @@
     <xacro:schunk_gripper hardware_interface="$(arg hardware_interface)" robot_name="$(arg gripper_name)">
     </xacro:schunk_gripper>
+    <xacro:implant_grasp_fingers gripper_name="$(arg gripper_name)"/>
     <joint name="milling_plate_base_joint" type="fixed">
         <parent link="optical_table_back_right_bolt"/>
@@ -51,3 +54,8 @@
     </joint>
     <xacro:cutting_plate />
+    <joint name="implant_a_joint" type="floating">
+        <parent link="world"/>
+        <child link="a_implant"/>
+    </joint>
+    <xacro:medpor_stock size="large" prefix="a"/>
 </robot>

File: ram_support/urdf/xacros/schunk_gripper.xacro (robot description, xacro)
@@ -23,5 +23,5 @@
       <origin xyz="-0.0058 0 0.0341" rpy="${pi/2} 0 -${pi/2}"/>
       <axis xyz="0 0 -1"/>
-      <limit lower="0.0" upper="0.005"
+      <limit lower="0.0008" upper="0.0058"
              effort="${max_effort}" velocity="0.0833" />
     </joint>
@@ -46,6 +46,7 @@
       <origin xyz="0.0058 0 0.0341" rpy="${pi/2} 0 ${pi/2}"/>
       <axis xyz="0 0 -1"/>
-      <limit lower="0.0" upper="0.005"
+      <limit lower="0.0008" upper="0.0058"
              effort="${max_effort}" velocity="0.0833" />
+      <mimic joint="${robot_name}_joint_left"/>
     </joint>
     <link name="${robot_name}_link_right">

Commit message: Added pykdl to install list and implant handler working with basic implementation

File: ram_support/urdf/mock_iiwa_workcell.urdf.xacro (robot description, xacro)
@@ -58,4 +58,10 @@
         <child link="a_implant"/>
     </joint>
+    <link name="home_a_implant"/>
+    <joint name="home_a_implant_joint" type="fixed">
+        <parent link="optical_table_back_left_bolt"/>
+        <child link="home_a_implant"/>
+        <origin xyz="0.5 -0.2 0.01" rpy="0.0 0.0 0"/>
+    </joint>
     <xacro:medpor_stock size="large" prefix="a"/>
 </robot>

File: ram_support/urdf/xacros/iiwa_14.xacro (robot description, xacro)
@@ -237,5 +237,5 @@
       <parent link="${robot_name}_link_6"/>
       <child link="${robot_name}_link_7"/>
-      <origin xyz="0 0 0" rpy="0 0 0"/>
+      <origin xyz="0 0 0" rpy="0 0 0"/>3BS
       <axis xyz="0 0 1"/>
       <limit lower="${-174 * PI / 180}" upper="${174 * PI / 180}"

Commit message: Have simulated gripper controller and implant handler for initial trajectory work

File: ram_support/urdf/mock_iiwa_workcell.urdf.xacro (robot description, xacro)
@@ -54,8 +54,4 @@
     </joint>
     <xacro:cutting_plate />
-    <joint name="implant_a_joint" type="floating">
-        <parent link="world"/>
-        <child link="a_implant"/>
-    </joint>
     <link name="home_a_implant"/>
     <joint name="home_a_implant_joint" type="fixed">
@@ -64,4 +60,3 @@
         <origin xyz="0.5 -0.2 0.01" rpy="0.0 0.0 0"/>
     </joint>
-    <xacro:medpor_stock size="large" prefix="a"/>
 </robot>

Commit message: toolpath follower working with the blade as a collision object, adding the blade as a touch link when required. cutting plate has been brought closer to the robot for the reach, should start testing with different positions of the cutting plate, maybe adding it as a virtual joint for ease

File: ram_support/urdf/mock_iiwa_workcell.urdf.xacro (robot description, xacro)
@@ -50,5 +50,5 @@
         <parent link="optical_table_front_right_bolt"/>
         <child link="cutting_plate"/>
-        <origin xyz="-0.2 0.2 0.00" rpy="0.0 0.0 0"/>
+        <origin xyz="-0.35 0.2 0.00" rpy="0.0 0.0 0"/>
     </joint>
     <xacro:cutting_plate />

Commit message: commented out changed cutting position, not working yet but needs to be looked into

File: ram_support/urdf/mock_iiwa_workcell.urdf.xacro (robot description, xacro)
@@ -50,5 +50,6 @@
         <parent link="optical_table_front_right_bolt"/>
         <child link="cutting_plate"/>
-        <origin xyz="-0.35 0.2 0.00" rpy="0.0 0.0 0"/>
+<!--        <origin xyz="0.0 0.2 0.30" rpy="0.0 -${pi/2} 0"/>-->
+        <origin xyz="-0.35 0.2 0.0" rpy="0 0 0"/>
     </joint>
     <xacro:cutting_plate />
@@ -57,5 +58,5 @@
         <parent link="optical_table_back_left_bolt"/>
         <child link="home_a_implant"/>
-        <origin xyz="0.5 -0.2 0.01" rpy="0.0 0.0 0"/>
+        <origin xyz="0.5 -0.2 0.01" rpy="0 0 0"/>
     </joint>
 </robot>
