Commit message: Moved to moveit2 and building

File: ram_support/urdf/iiwa_gripper.urdf.xacro (robot description, xacro)
@@ -6,9 +6,16 @@
     <xacro:include filename="$(find ram_support)/urdf/iiwa14.xacro"/>
     <xacro:include filename="$(find ram_support)/urdf/schunk_gripper.xacro"/>
+    <xacro:include filename="$(find ram_support)/urdf/optical_table.xacro"/>
     <xacro:arg name="iiwa_name" default="iiwa"/>
     <xacro:arg name="gripper_name" default="gripper"/>
     <xacro:arg name="hardware_interface" default="PositionJointInterface"/>
-    <joint name="$(arg iiwa_name)_world_joint" type="fixed">
+    <joint name="optical_table_world_joint" type="fixed">
         <parent link="world"/>
+        <child link="optical_table"/>
+        <origin xyz="0.0 0.0 0.006" rpy="0.0 0.0 ${pi/2}"/>
+    </joint>
+    <xacro:optical_table />
+    <joint name="$(arg iiwa_name)_base_joint" type="fixed">
+        <parent link="optical_table_front_left_bolt"/>
         <child link="$(arg iiwa_name)_link_0"/>
         <origin xyz="0.0 0.0 0.006" rpy="0.0 0.0 ${pi/2}"/>

Commit message: Setup small test workcell with iiwa, gripper, cutting table and milling table

File: ram_support/urdf/iiwa_gripper.urdf.xacro (robot description, xacro)
@@ -4,13 +4,27 @@
     <xacro:arg name="initial_z" default="0.0"/>
     <link name="world"/>
-    <xacro:include filename="$(find ram_support)/urdf/iiwa14.xacro"/>
-    <xacro:include filename="$(find ram_support)/urdf/schunk_gripper.xacro"/>
+    <xacro:include filename="$(find ram_support)/urdf/xacros/iiwa_14.xacro"/>
+    <xacro:include filename="$(find ram_support)/urdf/xacros/schunk_gripper.xacro"/>
+    <xacro:include filename="$(find ram_support)/urdf/xacros/optical_table.xacro"/>
+    <xacro:include filename="$(find ram_support)/urdf/xacros/iiwa_14_mounting_plate.xacro"/>
     <xacro:arg name="iiwa_name" default="iiwa"/>
     <xacro:arg name="gripper_name" default="gripper"/>
     <xacro:arg name="hardware_interface" default="PositionJointInterface"/>
-    <joint name="$(arg iiwa_name)_world_joint" type="fixed">
+    <joint name="optical_table_world_joint" type="fixed">
         <parent link="world"/>
+        <child link="optical_table"/>
+        <origin xyz="0.0 0.0 0.006" rpy="0.0 0.0 ${pi/2}"/>
+    </joint>
+    <xacro:optical_table />
+    <joint name="$(arg iiwa_name)_mounting_plate_base_joint" type="fixed">
+        <parent link="optical_table_front_left_bolt"/>
+        <child link="$(arg iiwa_name)_mounting_plate_front_left_bolt"/>
+        <origin xyz="0.175 0.150 0.00" rpy="0.0 0.0 0"/>
+    </joint>
+    <xacro:iiwa_14_mounting_plate robot_name="$(arg iiwa_name)"/>
+    <joint name="$(arg iiwa_name)_base_joint" type="fixed">
+        <parent link="$(arg iiwa_name)_mounting_plate_centre_top_surface"/>
         <child link="$(arg iiwa_name)_link_0"/>
-        <origin xyz="0.0 0.0 0.006" rpy="0.0 0.0 ${pi/2}"/>
+        <origin xyz="0 0 0" rpy="0.0 0.0 ${pi}"/>
     </joint>
     <xacro:iiwa14 hardware_interface="$(arg hardware_interface)" robot_name="$(arg iiwa_name)">
@@ -19,5 +33,5 @@
         <parent link="$(arg iiwa_name)_link_ee"/>
         <child link="$(arg gripper_name)_link_main_body"/>
-        <origin xyz="0.0 0.0 0.006" rpy="0.0 0.0 0"/>
+        <origin xyz="0 0 0.006" rpy="0.0 0.0 ${pi/2}"/>
     </joint>
     <xacro:schunk_gripper hardware_interface="$(arg hardware_interface)" robot_name="$(arg gripper_name)">

File: ram_support/urdf/xacros/iiwa_14.xacro (robot description, xacro)
@@ -2,5 +2,5 @@
 <robot xmlns:xacro="http://www.ros.org/wiki/xacro">
   <!-- Import Transmissions -->
-  <xacro:include filename="$(find ram_support)/urdf/iiwa.transmission.xacro" />
+  <xacro:include filename="$(find ram_support)/urdf/xacros/iiwa.transmission.xacro" />
   <!-- some constants -->
   <xacro:property name="safety_controller_k_pos" value="10" /> <!-- This sets the velocity according the distance the soft limits, velocity = -k_pos * (pos - soft_limit) -->
@@ -39,5 +39,5 @@
       <parent link="${robot_name}_link_0"/>
       <child link="${robot_name}_link_1"/>
-      <origin xyz="0 0 0.1575" rpy="0 0 0"/>
+      <origin xyz="0 0 0" rpy="0 0 0" />
       <axis xyz="0 0 1"/>
       <limit lower="${-169 * PI / 180}" upper="${169 * PI / 180}"
@@ -72,6 +72,6 @@
       <parent link="${robot_name}_link_1"/>
       <child link="${robot_name}_link_2"/>
-      <origin xyz="0 0 0.2025" rpy="${PI / 2}   0 ${PI}"/>
-      <axis xyz="0 0 1"/>
+      <origin xyz="-0.00043624 0 0.36" rpy="0 0 0" />
+      <axis xyz="0 1 0"/>
       <limit lower="${-119 * PI / 180}" upper="${119 * PI / 180}"
              effort="${max_effort}" velocity="${85 * PI / 180}" />
@@ -105,5 +105,5 @@
       <parent link="${robot_name}_link_2"/>
       <child link="${robot_name}_link_3"/>
-      <origin xyz="0 0.2045 0" rpy="${PI / 2} 0 ${PI}"/>
+      <origin xyz="0 0 0" rpy="0 0 0" />
       <axis xyz="0 0 1"/>
       <limit lower="${-169 * PI / 180}" upper="${169 * PI / 180}"
@@ -138,6 +138,6 @@
       <parent link="${robot_name}_link_3"/>
       <child link="${robot_name}_link_4"/>
-      <origin xyz="0 0 0.2155" rpy="${PI / 2} 0 0"/>
-      <axis xyz="0 0 1"/>
+      <origin xyz="0.00043624 0 0.42" rpy="0 0 0" />
+      <axis xyz="0 -1 0"/>
       <limit lower="${-119 * PI / 180}" upper="${119 * PI / 180}"
              effort="${max_effort}" velocity="${75 * PI / 180}" />
@@ -171,5 +171,5 @@
       <parent link="${robot_name}_link_4"/>
       <child link="${robot_name}_link_5"/>
-      <origin xyz="0 0.1845 0" rpy="${-PI / 2} ${PI} 0"/>
+      <origin xyz="0 0 0" rpy="0 0 0" />
       <axis xyz="0 0 1"/>
       <limit lower="${-169 * PI / 180}" upper="${169 * PI / 180}"
@@ -204,6 +204,6 @@
       <parent link="${robot_name}_link_5"/>
       <child link="${robot_name}_link_6"/>
-      <origin xyz="0 0 0.2155" rpy="${PI / 2} 0 0"/>
-      <axis xyz="0 0 1"/>
+      <origin xyz="0 0 0.4" rpy="0 0 0" />
+      <axis xyz="0 1 0"/>
       <limit lower="${-119 * PI / 180}" upper="${119 * PI / 180}"
              effort="${max_effort}" velocity="${135 * PI / 180}" />
@@ -237,5 +237,5 @@
       <parent link="${robot_name}_link_6"/>
       <child link="${robot_name}_link_7"/>
-      <origin xyz="0 0.081 0" rpy="${- PI / 2} ${PI} 0"/>
+      <origin xyz="0 0 0" rpy="0 0 0"/>
       <axis xyz="0 0 1"/>
       <limit lower="${-174 * PI / 180}" upper="${174 * PI / 180}"
@@ -269,5 +269,5 @@
       <parent link="${robot_name}_link_7"/>
       <child link="${robot_name}_link_ee"/>
-      <origin xyz="0 0 0.045" rpy="0 0 0"/>
+      <origin xyz="0 0 0.126" rpy="0 0 0"/>
     </joint>
     <link name="${robot_name}_link_ee">

File: ram_support/urdf/xacros/schunk_gripper.xacro (robot description, xacro)
@@ -13,5 +13,5 @@
         <origin xyz="0 0 0" rpy="0 0 0"/>
         <geometry>
-          <mesh filename="package://ram_support/meshes/schunk_gripper/collision/main_body.stl"/>
+          <mesh filename="package://ram_support/meshes/schunk_gripper/collision/main_body.stl" scale="0.001 0.001 0.001"/>
         </geometry>
       </collision>
@@ -21,6 +21,6 @@
       <parent link="${robot_name}_link_main_body"/>
       <child link="${robot_name}_link_left"/>
-      <origin xyz="0 0 0.1575" rpy="0 0 0"/>
-      <axis xyz="1 0 0"/>
+      <origin xyz="-0.0058 0 0.0341" rpy="${pi/2} 0 -${pi/2}"/>
+      <axis xyz="0 0 -1"/>
       <limit lower="0.0" upper="0.005"
              effort="${max_effort}" velocity="0.0833" />
@@ -30,5 +30,5 @@
         <origin xyz="0 0 0" rpy="0 0 0"/>
         <geometry>
-          <mesh filename="package://ram_support/meshes/schunk_gripper/visual/jaw_left.dae"/>
+          <mesh filename="package://ram_support/meshes/schunk_gripper/visual/left_gripper.dae"/>
         </geometry>
       </visual>
@@ -36,5 +36,5 @@
         <origin xyz="0 0 0" rpy="0 0 0"/>
         <geometry>
-          <mesh filename="package://ram_support/meshes/schunk_gripper/collision/jaw_left.stl"/>
+          <mesh filename="package://ram_support/meshes/schunk_gripper/collision/left_gripper.stl" scale="0.001 0.001 0.001"/>
         </geometry>
       </collision>
@@ -44,6 +44,6 @@
       <parent link="${robot_name}_link_main_body"/>
       <child link="${robot_name}_link_right"/>
-      <origin xyz="0 0 0.1575" rpy="0 0 0"/>
-      <axis xyz="1 0 0"/>
+      <origin xyz="0.0058 0 0.0341" rpy="${pi/2} 0 ${pi/2}"/>
+      <axis xyz="0 0 -1"/>
       <limit lower="0.0" upper="0.005"
              effort="${max_effort}" velocity="0.0833" />
@@ -53,5 +53,5 @@
         <origin xyz="0 0 0" rpy="0 0 0"/>
         <geometry>
-          <mesh filename="package://ram_support/meshes/schunk_gripper/visual/jaw_right.dae"/>
+          <mesh filename="package://ram_support/meshes/schunk_gripper/visual/right_gripper.dae"/>
         </geometry>
       </visual>
@@ -59,5 +59,5 @@
         <origin xyz="0 0 0" rpy="0 0 0"/>
         <geometry>
-          <mesh filename="package://ram_support/meshes/schunk_gripper/collision/jaw_right.stl"/>
+          <mesh filename="package://ram_support/meshes/schunk_gripper/collision/right_gripper.stl" scale="0.001 0.001 0.001"/>
         </geometry>
       </collision>

Commit message: updated gripper to PGN-80 and started to implement basic stock material handler, currently immediately sets the stock implant to attached to the gripper

File: ram_support/urdf/iiwa_gripper.urdf.xacro (robot description, xacro)
@@ -5,5 +5,5 @@
     <link name="world"/>
     <xacro:include filename="$(find ram_support)/urdf/xacros/iiwa_14.xacro"/>
-    <xacro:include filename="$(find ram_support)/urdf/xacros/schunk_gripper.xacro"/>
+    <xacro:include filename="$(find ram_support)/urdf/xacros/schunk_gripper_pgn_100.xacro"/>
     <xacro:include filename="$(find ram_support)/urdf/xacros/optical_table.xacro"/>
     <xacro:include filename="$(find ram_support)/urdf/xacros/iiwa_14_mounting_plate.xacro"/>

File: ram_support/urdf/mock_iiwa_workcell.urdf.xacro (robot description, xacro)
@@ -5,10 +5,9 @@
     <link name="world"/>
     <xacro:include filename="$(find ram_support)/urdf/xacros/iiwa_14.xacro"/>
-    <xacro:include filename="$(find ram_support)/urdf/xacros/schunk_gripper.xacro"/>
+    <xacro:include filename="$(find ram_support)/urdf/xacros/schunk_gripper_pgn_80.xacro"/>
     <xacro:include filename="$(find ram_support)/urdf/xacros/optical_table.xacro"/>
     <xacro:include filename="$(find ram_support)/urdf/xacros/iiwa_14_mounting_plate.xacro"/>
     <xacro:include filename="$(find ram_support)/urdf/xacros/milling_plate.xacro"/>
     <xacro:include filename="$(find ram_support)/urdf/xacros/cutting_plate.xacro"/>
-    <xacro:include filename="$(find ram_support)/urdf/xacros/implant_grasp_fingers.xacro"/>
     <xacro:include filename="$(find ram_support)/urdf/xacros/medpor_stock.xacro"/>
     <xacro:arg name="iiwa_name" default="iiwa"/>
@@ -41,11 +40,11 @@
     <xacro:schunk_gripper hardware_interface="$(arg hardware_interface)" robot_name="$(arg gripper_name)">
     </xacro:schunk_gripper>
-    <xacro:implant_grasp_fingers gripper_name="$(arg gripper_name)"/>
-    <joint name="milling_plate_base_joint" type="fixed">
-        <parent link="optical_table_back_right_bolt"/>
-        <child link="milling_plate"/>
-        <origin xyz="-0.2 -0.2 0.00" rpy="0.0 0.0 0"/>
-    </joint>
-    <xacro:milling_plate tool_length="0.005" tool_diameter="0.002"/>
+<!--    <xacro:implant_grasp_fingers gripper_name="$(arg gripper_name)"/>-->
+<!--    <joint name="milling_plate_base_joint" type="fixed">-->
+<!--        <parent link="optical_table_back_right_bolt"/>-->
+<!--        <child link="milling_plate"/>-->
+<!--        <origin xyz="-0.2 -0.2 0.00" rpy="0.0 0.0 0"/>-->
+<!--    </joint>-->
+<!--    <xacro:milling_plate tool_length="0.005" tool_diameter="0.002"/>-->
     <joint name="cutting_plate_base_joint" type="fixed">
         <parent link="optical_table_front_right_bolt"/>

File: ram_support/urdf/xacros/schunk_gripper_pgn_80.xacro (robot description, xacro)
@@ -7,5 +7,5 @@
         <origin xyz="0 0 0" rpy="0 0 0"/>
         <geometry>
-          <mesh filename="package://ram_support/meshes/schunk_gripper/visual/main_body.dae"/>
+          <mesh filename="package://ram_support/meshes/schunk_gripper/pgn_80/visual/SCHUNK_PGN-plus-P_80-2_mainbody.dae"/>
         </geometry>
       </visual>
@@ -13,5 +13,5 @@
         <origin xyz="0 0 0" rpy="0 0 0"/>
         <geometry>
-          <mesh filename="package://ram_support/meshes/schunk_gripper/collision/main_body.stl" scale="0.001 0.001 0.001"/>
+          <mesh filename="package://ram_support/meshes/schunk_gripper/pgn_80/collision/SCHUNK_PGN-plus-P_80-2_mainbody.stl"/>
         </geometry>
       </collision>
@@ -21,7 +21,6 @@
       <parent link="${robot_name}_link_main_body"/>
       <child link="${robot_name}_link_left"/>
-      <origin xyz="-0.0058 0 0.0341" rpy="${pi/2} 0 -${pi/2}"/>
-      <axis xyz="0 0 -1"/>
-      <limit lower="0.0008" upper="0.0058"
+      <origin xyz="0 0 0.0" rpy="0 0 0"/>
+      <limit lower="0.000" upper="0.005"
              effort="${max_effort}" velocity="0.0833" />
     </joint>
@@ -30,5 +29,5 @@
         <origin xyz="0 0 0" rpy="0 0 0"/>
         <geometry>
-          <mesh filename="package://ram_support/meshes/schunk_gripper/visual/left_gripper.dae"/>
+          <mesh filename="package://ram_support/meshes/schunk_gripper/pgn_80/visual/SCHUNK_PGN-plus-P_80-2_jaw.dae"/>
         </geometry>
       </visual>
@@ -36,5 +35,5 @@
         <origin xyz="0 0 0" rpy="0 0 0"/>
         <geometry>
-          <mesh filename="package://ram_support/meshes/schunk_gripper/collision/left_gripper.stl" scale="0.001 0.001 0.001"/>
+          <mesh filename="package://ram_support/meshes/schunk_gripper/pgn_80/collision/SCHUNK_PGN-plus-P_80-2_jaw.stl" />
         </geometry>
       </collision>
@@ -44,7 +43,7 @@
       <parent link="${robot_name}_link_main_body"/>
       <child link="${robot_name}_link_right"/>
-      <origin xyz="0.0058 0 0.0341" rpy="${pi/2} 0 ${pi/2}"/>
-      <axis xyz="0 0 -1"/>
-      <limit lower="0.0008" upper="0.0058"
+      <origin xyz="0 0 0" rpy="0 0 ${pi}"/>
+      <axis xyz="1 0 0"/>
+      <limit lower="0.000" upper="0.005"
              effort="${max_effort}" velocity="0.0833" />
       <mimic joint="${robot_name}_joint_left"/>
@@ -54,5 +53,5 @@
         <origin xyz="0 0 0" rpy="0 0 0"/>
         <geometry>
-          <mesh filename="package://ram_support/meshes/schunk_gripper/visual/right_gripper.dae"/>
+          <mesh filename="package://ram_support/meshes/schunk_gripper/pgn_80/visual/SCHUNK_PGN-plus-P_80-2_jaw.dae"/>
         </geometry>
       </visual>
@@ -60,5 +59,5 @@
         <origin xyz="0 0 0" rpy="0 0 0"/>
         <geometry>
-          <mesh filename="package://ram_support/meshes/schunk_gripper/collision/right_gripper.stl" scale="0.001 0.001 0.001"/>
+          <mesh filename="package://ram_support/meshes/schunk_gripper/pgn_80/collision/SCHUNK_PGN-plus-P_80-2_jaw.stl"/>
         </geometry>
       </collision>

Commit message: Remade model for actual setup

File: ram_support/urdf/iiwa_gripper.urdf.xacro (robot description, xacro)
@@ -5,5 +5,5 @@
     <link name="world"/>
     <xacro:include filename="$(find ram_support)/urdf/xacros/iiwa_14.xacro"/>
-    <xacro:include filename="$(find ram_support)/urdf/xacros/schunk_gripper_pgn_100.xacro"/>
+    <xacro:include filename="$(find ram_support)/urdf/xacros/schunk_gripper_pgn_80.xacro"/>
     <xacro:include filename="$(find ram_support)/urdf/xacros/optical_table.xacro"/>
     <xacro:include filename="$(find ram_support)/urdf/xacros/iiwa_14_mounting_plate.xacro"/>
@@ -31,7 +31,8 @@
     </xacro:iiwa14>
     <joint name="$(arg iiwa_name)_to_$(arg gripper_name)_joint" type="fixed">
-        <parent link="$(arg iiwa_name)_link_ee"/>
-        <child link="$(arg gripper_name)_link_main_body"/>
-        <origin xyz="0 0 0.006" rpy="0.0 0.0 ${pi/2}"/>
+<!--        <parent link="$(arg iiwa_name)_link_ee"/>-->
+        <parent link="world"/>
+        <child link="$(arg gripper_name)_link_iiwa_attachment"/>
+        <origin xyz="0 0 0.00" rpy="0.0 0.0 0.0"/> <!-- ${pi/2} -->
     </joint>
     <xacro:schunk_gripper hardware_interface="$(arg hardware_interface)" robot_name="$(arg gripper_name)">

File: ram_support/urdf/mock_iiwa_workcell.urdf.xacro (robot description, xacro)
@@ -23,5 +23,5 @@
         <parent link="optical_table_front_left_bolt"/>
         <child link="$(arg iiwa_name)_mounting_plate_front_left_bolt"/>
-        <origin xyz="0.175 0.150 0.00" rpy="0.0 0.0 0"/>
+        <origin xyz="0.125 0.125 0.00" rpy="0.0 0.0 0"/>
     </joint>
     <xacro:iiwa_14_mounting_plate robot_name="$(arg iiwa_name)"/>
@@ -35,6 +35,6 @@
     <joint name="$(arg iiwa_name)_to_$(arg gripper_name)_joint" type="fixed">
         <parent link="$(arg iiwa_name)_link_ee"/>
-        <child link="$(arg gripper_name)_link_main_body"/>
-        <origin xyz="0 0 0.006" rpy="0.0 0.0 ${pi/2}"/>
+        <child link="$(arg gripper_name)_link_iiwa_attachment"/>
+        <origin xyz="0 0 0.00" rpy="0 0 -${pi/2}"/>
     </joint>
     <xacro:schunk_gripper hardware_interface="$(arg hardware_interface)" robot_name="$(arg gripper_name)">

File: ram_support/urdf/xacros/schunk_gripper_pgn_80.xacro (robot description, xacro)
@@ -3,4 +3,23 @@
   <xacro:property name="max_effort" value="300"/> <!-- Should be changed to match the robots specs -->
   <xacro:macro name="schunk_gripper" params="hardware_interface robot_name">
+    <link name="${robot_name}_link_iiwa_attachment">
+      <visual>
+        <origin xyz="0 0 0" rpy="0 0 0"/>
+        <geometry>
+          <mesh filename="package://ram_support/meshes/schunk_gripper/pgn_80/visual/gripper_iiwa_attachment.dae"/>
+        </geometry>
+      </visual>
+      <collision>
+        <origin xyz="0 0 0" rpy="0 0 0"/>
+        <geometry>
+          <mesh filename="package://ram_support/meshes/schunk_gripper/pgn_80/collision/gripper_iiwa_attachment.stl"/>
+        </geometry>
+      </collision>
+    </link>
+    <joint name="${robot_name}_iiwa_attachment_joint" type="fixed">
+      <parent link="${robot_name}_link_iiwa_attachment"/>
+      <child link="${robot_name}_link_main_body"/>
+      <origin xyz="0 0 0.0195" rpy="0 0 -${pi/4}"/>
+    </joint>
     <link name="${robot_name}_link_main_body">
       <visual>
