Commit message: made iiwa_workcell file with profile us cutter enclosure and actual gripper attachment

File: ram_support/urdf/iiwa_workcell.urdf.xacro (robot description, xacro)
@@ -8,6 +8,5 @@
     <xacro:include filename="$(find ram_support)/urdf/xacros/optical_table.xacro"/>
     <xacro:include filename="$(find ram_support)/urdf/xacros/iiwa_14_mounting_plate.xacro"/>
-    <xacro:include filename="$(find ram_support)/urdf/xacros/milling_plate.xacro"/>
-    <xacro:include filename="$(find ram_support)/urdf/xacros/mock_cutting_plate.xacro"/>
+    <xacro:include filename="$(find ram_support)/urdf/xacros/cutting_plate.xacro"/>
     <xacro:include filename="$(find ram_support)/urdf/xacros/medpor_stock.xacro"/>
     <xacro:arg name="iiwa_name" default="iiwa"/>
@@ -23,5 +22,5 @@
         <parent link="optical_table_front_left_bolt"/>
         <child link="$(arg iiwa_name)_mounting_plate_front_left_bolt"/>
-        <origin xyz="0.125 0.125 0.00" rpy="0.0 0.0 0"/>
+        <origin xyz="0.175 0.150 0.00" rpy="0.0 0.0 0"/>
     </joint>
     <xacro:iiwa_14_mounting_plate robot_name="$(arg iiwa_name)"/>
@@ -40,16 +39,9 @@
     <xacro:schunk_gripper hardware_interface="$(arg hardware_interface)" robot_name="$(arg gripper_name)">
     </xacro:schunk_gripper>
-<!--    <xacro:implant_grasp_fingers gripper_name="$(arg gripper_name)"/>-->
-<!--    <joint name="milling_plate_base_joint" type="fixed">-->
-<!--        <parent link="optical_table_back_right_bolt"/>-->
-<!--        <child link="milling_plate"/>-->
-<!--        <origin xyz="-0.2 -0.2 0.00" rpy="0.0 0.0 0"/>-->
-<!--    </joint>-->
-<!--    <xacro:milling_plate tool_length="0.005" tool_diameter="0.002"/>-->
     <joint name="cutting_plate_base_joint" type="fixed">
-        <parent link="optical_table_front_right_bolt"/>
+        <parent link="optical_table_back_left_bolt"/>
         <child link="cutting_plate"/>
 <!--        <origin xyz="0.0 0.2 0.30" rpy="0.0 -${pi/2} 0"/>-->
-        <origin xyz="-0.35 0.2 0.0" rpy="0 0 0"/>
+        <origin xyz="-0.17351 -0.237 0.051" rpy="0 0 0"/>
     </joint>
     <xacro:cutting_plate />

File: ram_support/urdf/xacros/mock_cutting_plate.xacro (robot description, xacro)
@@ -6,11 +6,11 @@
         <origin xyz="0 0 0" rpy="0 0 0"/>
         <geometry>
-          <mesh filename="package://ram_support/meshes/tools/visual/us_cutter_enclosure.dae"/>
+          <mesh filename="package://ram_support/meshes/tools/visual/mock_cutting_plate.dae"/>
         </geometry>
       </visual>
       <collision>
-        <origin xyz="0 0 0" rpy="0 0 ${-pi/2}"/>
+        <origin xyz="0 0 0.125" rpy="0 0 0"/>
         <geometry>
-          <mesh filename="package://ram_support/meshes/tools/collision/us_cutter_enclosure.stl"/>
+          <box size="0.25 0.25 0.25"/>
         </geometry>
       </collision>
@@ -19,5 +19,5 @@
       <parent link="cutting_plate"/>
       <child link="cutting_plate_base"/>
-      <origin xyz="0 0 0" rpy="0 0 0"/>
+      <origin xyz="0 0 0.25" rpy="0 0 0"/>
     </joint>
     <link name="cutting_plate_base"/>
@@ -42,5 +42,5 @@
       <parent link="cutting_plate_base"/>
       <child link="cutting_tool"/>
-      <origin xyz="0.017 0 -0.0035" rpy="0 0 0"/>
+      <origin xyz="0 0 -0.0035" rpy="0 0 0"/>
     </joint>
     <joint name="cutting_tool_base_joint" type="fixed">

Commit message: updated us_cutter enclosure model

File: ram_support/urdf/iiwa_workcell.urdf.xacro (robot description, xacro)
@@ -43,5 +43,5 @@
         <child link="cutting_plate"/>
 <!--        <origin xyz="0.0 0.2 0.30" rpy="0.0 -${pi/2} 0"/>-->
-        <origin xyz="-0.17351 -0.237 0.051" rpy="0 0 0"/>
+        <origin xyz="-0.17351 -0.237 0.108" rpy="0 0 0"/>
     </joint>
     <xacro:cutting_plate />

Commit message: Adjusting position of kuka to match hardware setup

File: ram_support/urdf/iiwa_workcell.urdf.xacro (robot description, xacro)
@@ -22,5 +22,5 @@
         <parent link="optical_table_front_left_bolt"/>
         <child link="$(arg iiwa_name)_mounting_plate_front_left_bolt"/>
-        <origin xyz="0.175 0.150 0.00" rpy="0.0 0.0 0"/>
+        <origin xyz="0.125 0.125 0.00" rpy="0.0 0.0 0"/>
     </joint>
     <xacro:iiwa_14_mounting_plate robot_name="$(arg iiwa_name)"/>

Commit message: modified height of cutting plate using the robot to calibrate

File: ram_support/urdf/iiwa_workcell.urdf.xacro (robot description, xacro)
@@ -43,5 +43,5 @@
         <child link="cutting_plate"/>
 <!--        <origin xyz="0.0 0.2 0.30" rpy="0.0 -${pi/2} 0"/>-->
-        <origin xyz="-0.17351 -0.237 0.108" rpy="0 0 0"/>
+        <origin xyz="-0.17351 -0.237 0.1109" rpy="0 0 0"/>
     </joint>
     <xacro:cutting_plate />

Commit message: Setting up implant holder urdf and paraming the blade height. Need to add allowed collision with implant support now

File: ram_support/urdf/iiwa_workcell.urdf.xacro (robot description, xacro)
@@ -1,6 +1,5 @@
 <?xml version="1.0"?>
 <robot xmlns:xacro="http://www.ros.org/wiki/xacro" name="iiwa_workcell">
-    <xacro:arg name="hardware_interface" default="PositionJointInterface"/>
-    <xacro:arg name="initial_z" default="0.0"/>
+    <xacro:arg name="blade_height" default="0.0025"/>
     <link name="world"/>
     <xacro:include filename="$(find ram_support)/urdf/xacros/iiwa_14.xacro"/>
@@ -45,5 +44,6 @@
         <origin xyz="-0.17351 -0.237 0.1109" rpy="0 0 0"/>
     </joint>
-    <xacro:cutting_plate />
+    <xacro:cutting_plate blade_height="$(arg blade_height)"/>
+<!--    <xacro:cutting_plate />-->
     <link name="home_a_implant"/>
     <joint name="home_a_implant_joint" type="fixed">

File: ram_support/urdf/xacros/cutting_plate.xacro (robot description, xacro)
@@ -1,5 +1,7 @@
 <?xml version="1.0"?>
 <robot xmlns:xacro="http://www.ros.org/wiki/xacro">
-  <xacro:macro name="cutting_plate">
+  <xacro:macro name="cutting_plate" params="blade_height:=^|0.0025">
+<!--    <xacro:arg name="blade_height" default="0.0025"/>-->
+    <xacro:property name="intersection_offset" value="0.00026" /> <!-- If there is a chisel tip this is the offset to the intersection point of the edges-->
     <link name="cutting_plate">
       <visual>
@@ -42,10 +44,10 @@
       <parent link="cutting_plate_base"/>
       <child link="cutting_tool"/>
-      <origin xyz="0.017 0 -0.0035" rpy="0 0 0"/>
+      <origin xyz="0.017 0 ${-0.0087 + blade_height}" rpy="0 0 0"/>
     </joint>
     <joint name="cutting_tool_base_joint" type="fixed">
       <parent link="cutting_tool"/>
       <child link="cutting_tool_base"/>
-      <origin xyz="-0.003152 0 0.0035" rpy="0 0 0"/>
+      <origin xyz="${(blade_height + intersection_offset) * tan(30 * pi / 180)} 0 ${0.0087 - blade_height}" rpy="0 0 0"/>
     </joint>
     <joint name="cutting_tool_tip_joint" type="fixed">

File: ram_support/urdf/xacros/schunk_gripper_pgn_80.xacro (robot description, xacro)
@@ -33,4 +33,42 @@
         <geometry>
           <mesh filename="package://ram_support/meshes/schunk_gripper/pgn_80/collision/SCHUNK_PGN-plus-P_80-2_mainbody.stl"/>
+        </geometry>
+      </collision>
+    </link>
+    <joint name="${robot_name}_joint_implant_holder" type="fixed">
+      <parent link="${robot_name}_link_main_body"/>
+      <child link="${robot_name}_implant_holder"/>
+      <origin xyz="0 0 0.0" rpy="0 0 0"/>
+    </joint>
+    <link name="${robot_name}_implant_holder">
+      <visual>
+        <origin xyz="0 0 0" rpy="0 0 0"/>
+        <geometry>
+          <mesh filename="package://ram_support/meshes/schunk_gripper/pgn_80/visual/implant_holder.dae"/>
+        </geometry>
+      </visual>
+      <collision>
+        <origin xyz="0 0 0" rpy="0 0 0"/>
+        <geometry>
+          <mesh filename="package://ram_support/meshes/schunk_gripper/pgn_80/collision/implant_holder.stl" />
+        </geometry>
+      </collision>
+    </link>
+    <joint name="${robot_name}_joint_implant_support" type="fixed">
+      <parent link="${robot_name}_link_main_body"/>
+      <child link="${robot_name}_implant_support"/>
+      <origin xyz="0 0 0.0" rpy="0 0 0"/>
+    </joint>
+    <link name="${robot_name}_implant_support">
+      <visual>
+        <origin xyz="0 0 0" rpy="0 0 0"/>
+        <geometry>
+          <mesh filename="package://ram_support/meshes/schunk_gripper/pgn_80/visual/implant_support.dae"/>
+        </geometry>
+      </visual>
+      <collision>
+        <origin xyz="0 0 0" rpy="0 0 0"/>
+        <geometry>
+          <mesh filename="package://ram_support/meshes/schunk_gripper/pgn_80/collision/implant_support.stl" />
         </geometry>
       </collision>
@@ -86,5 +124,5 @@
       <parent link="${robot_name}_link_main_body"/>
       <child link="${robot_name}_jaw_centre"/>
-      <origin xyz="0 0 0.078850" rpy="0 0 0"/>
+      <origin xyz="0 0 0.065850" rpy="0 0 0"/>
     </joint>
     <link name="${robot_name}_jaw_left"/>
@@ -92,5 +130,5 @@
       <parent link="${robot_name}_link_left"/>
       <child link="${robot_name}_jaw_left"/>
-      <origin xyz="0.000524 0 0.078850" rpy="0 0 0"/>
+      <origin xyz="0.000524 0 0.065850" rpy="0 0 0"/>
     </joint>
     <link name="${robot_name}_jaw_right"/>
@@ -98,5 +136,5 @@
       <parent link="${robot_name}_link_right"/>
       <child link="${robot_name}_jaw_right"/>
-      <origin xyz="0.000524 0 0.078850" rpy="0 0 ${pi}"/>
+      <origin xyz="0.000524 0 0.065850" rpy="0 0 ${pi}"/>
     </joint>
     <xacro:include filename="$(find ram_support)/urdf/xacros/control/gripper.ros2_control.xacro" />

Commit message: updated robot position on optical table

File: ram_support/urdf/iiwa_workcell.urdf.xacro (robot description, xacro)
@@ -21,5 +21,5 @@
         <parent link="optical_table_front_left_bolt"/>
         <child link="$(arg iiwa_name)_mounting_plate_front_left_bolt"/>
-        <origin xyz="0.125 0.125 0.00" rpy="0.0 0.0 0"/>
+        <origin xyz="0.025 0.025 0.00" rpy="0.0 0.0 0"/>
     </joint>
     <xacro:iiwa_14_mounting_plate robot_name="$(arg iiwa_name)"/>

Commit message: Adding cutting plate buffer object and modifying acm for planning. behaviour now launch with toolpath planner

File: ram_support/urdf/iiwa_workcell.urdf.xacro (robot description, xacro)
@@ -40,5 +40,5 @@
     <joint name="cutting_plate_base_joint" type="fixed">
         <parent link="optical_table_back_left_bolt"/>
-        <child link="cutting_plate"/>
+        <child link="us_cutter_enclosure"/>
 <!--        <origin xyz="0.0 0.2 0.30" rpy="0.0 -${pi/2} 0"/>-->
         <origin xyz="-0.17351 -0.237 0.1109" rpy="0 0 0"/>

File: ram_support/urdf/xacros/cutting_plate.xacro (robot description, xacro)
@@ -4,5 +4,5 @@
 <!--    <xacro:arg name="blade_height" default="0.0025"/>-->
     <xacro:property name="intersection_offset" value="0.00026" /> <!-- If there is a chisel tip this is the offset to the intersection point of the edges-->
-    <link name="cutting_plate">
+    <link name="us_cutter_enclosure">
       <visual>
         <origin xyz="0 0 0" rpy="0 0 0"/>
@@ -14,14 +14,27 @@
         <origin xyz="0 0 0" rpy="0 0 ${-pi/2}"/>
         <geometry>
-          <mesh filename="package://ram_support/meshes/tools/collision/us_cutter_enclosure.stl"/>
+          <mesh filename="package://ram_support/meshes/tools/collision/collision_us_cutter_enclosure.stl"/>
         </geometry>
       </collision>
     </link>
-    <joint name="cutting_plate_surface_joint" type="fixed">
-      <parent link="cutting_plate"/>
+    <link name="cutting_plate_base">
+<!--      <visual>-->
+<!--        <origin xyz="0 0 -0.005" rpy="0 0 0"/>-->
+<!--        <geometry>-->
+<!--            <box size="0.315 0.315 0.01" />-->
+<!--        </geometry>-->
+<!--      </visual>-->
+      <collision>
+        <origin xyz="0 0 -0.005" rpy="0 0 ${-pi/2}"/>
+        <geometry>
+            <box size="0.315 0.315 0.01" />
+        </geometry>
+      </collision>
+    </link>
+    <joint name="us_cutter_surface_joint" type="fixed">
+      <parent link="us_cutter_enclosure"/>
       <child link="cutting_plate_base"/>
       <origin xyz="0 0 0" rpy="0 0 0"/>
     </joint>
-    <link name="cutting_plate_base"/>
   <!-- Cutting tool selected-->
     <link name="cutting_tool">
