Commit message: Integration with ROS2 control and iiwa interface, fake is now handled by fakecomponents within ros2 control

File: ram_support/urdf/xacros/control/iiwa.ros2_control.xacro (robot description, xacro)
@@ -1,11 +1,11 @@
 <?xml version="1.0"?>
 <robot xmlns:xacro="http://www.ros.org/wiki/xacro">
-    <xacro:macro name="iiwa_position_only" params="name">
+    <xacro:macro name="iiwa_position_only" params="name robot_ip robot_port">
         <ros2_control name="${name}" type="system">
             <hardware>
-<!--                <plugin>iiwa_fri_ros/IiwaHWInterface</plugin>-->
-<!--                <param name="robot_ip">${robot_ip}</param>-->
-<!--                <param name="robot_port">${robot_port}</param>-->
-                <plugin>fake_components/GenericSystem</plugin>
+                <plugin>iiwa_fri_ros/IiwaHWInterface</plugin>
+                <param name="robot_ip">${robot_ip}</param>
+                <param name="robot_port">${robot_port}</param>
+<!--                <plugin>fake_components/GenericSystem</plugin>-->
             </hardware>
             <joint name="iiwa_joint_1">

File: ram_support/urdf/xacros/iiwa_14.xacro (robot description, xacro)
@@ -11,4 +11,6 @@
   <xacro:macro name="iiwa14" params="hardware_interface robot_name">
     <xacro:arg name="use_ros2_control" default="true"/>
+    <xacro:arg name="robot_ip" default="192.170.10.2"/>
+    <xacro:arg name="robot_port" default="30200"/>
     <link name="${robot_name}_link_0">
       <inertial>
@@ -277,7 +279,7 @@
     <xacro:if value="$(arg use_ros2_control)" >
       <xacro:include filename="$(find ram_support)/urdf/xacros/control/iiwa.ros2_control.xacro" />
-      <xacro:iiwa_position_only name="IiwaFakePositionHardwareInterface"/>
-<!--                                robot_ip="$(arg robot_ip)"-->
-<!--                                robot_port="$(arg robot_port)"/>-->
+      <xacro:iiwa_position_only name="IiwaFakePositionHardwareInterface"
+                                robot_ip="$(arg robot_ip)"
+                                robot_port="$(arg robot_port)"/>
     </xacro:if>
     <xacro:unless value="$(arg use_ros2_control)" >

Commit message: added hardware tag but not implemented in launch file yet

File: ram_support/urdf/xacros/control/iiwa.ros2_control.xacro (robot description, xacro)
@@ -1,11 +1,15 @@
 <?xml version="1.0"?>
 <robot xmlns:xacro="http://www.ros.org/wiki/xacro">
-    <xacro:macro name="iiwa_position_only" params="name robot_ip robot_port">
+    <xacro:macro name="iiwa_position_only" params="name robot_ip robot_port hardware:=false">
         <ros2_control name="${name}" type="system">
             <hardware>
-                <plugin>iiwa_fri_ros/IiwaHWInterface</plugin>
-                <param name="robot_ip">${robot_ip}</param>
-                <param name="robot_port">${robot_port}</param>
-<!--                <plugin>fake_components/GenericSystem</plugin>-->
+                <xacro:if value="${hardware}">
+                    <plugin>iiwa_fri_ros/IiwaHWInterface</plugin>
+                    <param name="robot_ip">${robot_ip}</param>
+                    <param name="robot_port">${robot_port}</param>
+                </xacro:if>
+                <xacro:unless value="${hardware}">
+                    <plugin>fake_components/GenericSystem</plugin>
+                </xacro:unless>
             </hardware>
             <joint name="iiwa_joint_1">

File: ram_support/urdf/xacros/iiwa_14.xacro (robot description, xacro)
@@ -1,6 +1,4 @@
 <?xml version="1.0"?>
 <robot xmlns:xacro="http://www.ros.org/wiki/xacro">
-  <!-- Import Transmissions -->
-  <xacro:include filename="$(find ram_support)/urdf/xacros/iiwa.transmission.xacro" />
   <!-- some constants -->
   <xacro:property name="safety_controller_k_pos" value="10" /> <!-- This sets the velocity according the distance the soft limits, velocity = -k_pos * (pos - soft_limit) -->
@@ -13,4 +11,5 @@
     <xacro:arg name="robot_ip" default="192.170.10.2"/>
     <xacro:arg name="robot_port" default="30200"/>
+    <xacro:arg name="hardware" default="false"/>
     <link name="${robot_name}_link_0">
       <inertial>
@@ -279,9 +278,11 @@
     <xacro:if value="$(arg use_ros2_control)" >
       <xacro:include filename="$(find ram_support)/urdf/xacros/control/iiwa.ros2_control.xacro" />
-      <xacro:iiwa_position_only name="IiwaFakePositionHardwareInterface"
+      <xacro:iiwa_position_only name="IiwaPositionHardwareInterface"
                                 robot_ip="$(arg robot_ip)"
-                                robot_port="$(arg robot_port)"/>
+                                robot_port="$(arg robot_port)"
+                                hardware="$(arg hardware)"/>
     </xacro:if>
     <xacro:unless value="$(arg use_ros2_control)" >
+      <xacro:include filename="$(find ram_support)/urdf/xacros/iiwa.transmission.xacro" />
       <xacro:iiwa_transmission hardware_interface="${hardware_interface}" robot_name="${robot_name}"/>
     </xacro:unless>
